Commit message: Auto commit for 2024-09-16

File: src/learning_urdf_rviz_gazebo/urdf/urdf/demo05_test.urdf (robot description, URDF)
Before this commit: robot mycar, 1 links, 0 joints
Links:
- added link back_wheel; visual sphere radius=0.0075
- added link base_link; visual cylinder length=0.08 radius=0.1
- added link front_wheel; visual sphere radius=0.0075
- added link left_wheel; visual cylinder length=0.015 radius=0.0325
- added link right_wheel; visual cylinder length=0.015 radius=0.0325
Joints:
- added joint back_wheel2base_link: type continuous, parent base_link, child back_wheel, origin xyz=-0.0925 0 -0.0475, axis 1 1 1
- added joint base_link2base_footprint: type fixed, parent base_footprint, child base_link, origin xyz=0 0 0.055 rpy=0 0 0
- added joint front_wheel2base_link: type continuous, parent base_link, child front_wheel, origin xyz=0.0925 0 -0.0475, axis 1 1 1
- added joint left_wheel2base_link: type continuous, parent base_link, child left_wheel, origin xyz=0 0.1 -0.0225, axis 0 1 0
- added joint right_wheel2base_link: type continuous, parent base_link, child right_wheel, origin xyz=0 -0.1 -0.0225, axis 0 1 0
